File: schema.kicad_sch (KiCad schematic)
At the start: 5 parts, among them U1 74HC595D, U2 74HC595D, U5 28C256

Commit message: fix-wrong-zif
Parts:
- U5: value 28C256 -> AT28C256-15PU; footprint Socket:DIP_Socket-24_W11.9_W12.7_W15.24_W17.78_W18.5_3M_224-1275-00-0602J -> Socket:DIP_Socket-28_W11.9_W12.7_W15.24_W17.78_W18.5_3M_228-1277-00-0602J
Changed lines of the file:
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@@
     (title "Erinnerlichkeit")
     (date "2024-04-22")
-    (rev "0.0.2")
+    (rev "0.0.3")
     (company "Entropia e.V.")
     (comment 1 "@proliecan@chaos.social")
@@
       (effects (font (size 1.27 1.27)) (justify left))
     )
-    (property "Value" "28C256" (at 116.4941 26.67 0)
-      (effects (font (size 1.27 1.27)) (justify left))
-    )
-    (property "Footprint" "Socket:DIP_Socket-24_W11.9_W12.7_W15.24_W17.78_W18.5_3M_224-1275-00-0602J" (at 114.3 54.61 0)
-      (effects (font (size 1.27 1.27)) hide)
-    )
+    (property "Value" "AT28C256-15PU" (at 116.4941 26.67 0)
+      (effects (font (size 1.27 1.27)) (justify left))
+    )
+    (property "Footprint" "Socket:DIP_Socket-28_W11.9_W12.7_W15.24_W17.78_W18.5_3M_228-1277-00-0602J" (at 114.3 54.61 0)
+      (effects (font (size 1.27 1.27)) hide)
+    )
